Commit message: Created Gazebo model and world

File: description/robot.urdf.xacro (robot description, xacro)
@@ -1,4 +1,5 @@
 <?xml version="1.0"?>
 <robot xmlns:xacro="http://www.ros.org/wiki/xacro"  name="robot">
-  <xacro:include filename="robot_core.xacro" />
+    <xacro:include filename="robot_core.xacro" />
+    <xacro:include filename="gazebo_control.xacro" />
 </robot>

File: description/robot_core.xacro (robot description, xacro)
@@ -41,4 +41,7 @@
         </xacro:inertial_box>
    </link>
+   <gazebo reference = "chassis">
+        <material>Gazebo/White</material>
+   </gazebo>
    <!-- Left Wheel link-->
    <joint name="left_wheel_joint" type="continuous">
@@ -64,4 +67,7 @@
         </xacro:inertial_cylinder>
    </link>
+    <gazebo reference = "left_wheel">
+        <material>Gazebo/Blue</material>
+    </gazebo>
    <!-- Right Wheel link-->
    <joint name="right_wheel_joint" type="continuous">
@@ -70,21 +76,24 @@
     <origin xyz="0 -0.175 0 " rpy = "${pi/2} 0 0"/>
     <axis xyz = "0 0 -1"/>
-</joint>
-<link name="right_wheel">
-    <visual>
+    </joint>
+    <link name="right_wheel">
+        <visual>
+            <geometry>
+                <cylinder radius ="0.05" length ="0.04"/>
+            </geometry>
+            <material name = "blue"/>
+        </visual>
+        <collision>
         <geometry>
             <cylinder radius ="0.05" length ="0.04"/>
         </geometry>
-        <material name = "blue"/>
-    </visual>
-    <collision>
-        <geometry>
-            <cylinder radius ="0.05" length ="0.04"/>
-        </geometry>
-    </collision>
-    <xacro:inertial_cylinder mass="0.1" radius="0.05" length="0.04">
-        <origin xyz="0 0 0 " rpy = "0 0 0 "/>
-    </xacro:inertial_cylinder>
-</link>
+        </collision>
+        <xacro:inertial_cylinder mass="0.1" radius="0.05" length="0.04">
+            <origin xyz="0 0 0 " rpy = "0 0 0 "/>
+        </xacro:inertial_cylinder>
+    </link>
+    <gazebo reference = "right_wheel">
+        <material>Gazebo/Blue</material>
+    </gazebo>
     <!-- Caster Wheel Link-->
     <joint name="caster_wheel_joint" type="fixed">
@@ -109,3 +118,8 @@
         </xacro:inertial_sphere>
     </link>
+    <gazebo reference = "caster_wheel">
+        <material>Gazebo/Black</material>
+        <mu1 value = "0.001"/>
+        <mu2 value = "0.001"/>
+    </gazebo>
 </robot>
